Commit message: Second

File: Intermedio/urdf/phantom_1.xacro (robot description, xacro)
@@ -7,5 +7,5 @@
   AUTHORS: GUSTAVO ADOLFO BERDUGO VELASQUEZ, JUAN SEBASTIAN HERNANDEZ REYES
   -->
-<robot name="phantomXPincher1" xmlns:xacro="http://www.ros.org/wiki/xacro">
+<robot name="phantomXPincher" xmlns:xacro="http://www.ros.org/wiki/xacro">
   <!-- Include -->
   <xacro:include filename="$(find intermedio)/urdf/phantom_links-joints.xacro" />

File: Intermedio/urdf/phantom_parameters1.xacro (robot description, xacro)
@@ -1,16 +1,16 @@
 <?xml version="1.0" ?>
  <robot xmlns:xacro="http://www.ros.org/wiki/xacro">
- <xacro:property name="link_00_name" value="base_link_1" />
- <xacro:property name="link_01_name" value="link1_1" />
- <xacro:property name="link_02_name" value="link2_1" />
- <xacro:property name="link_03_name" value="link3_1" />
- <xacro:property name="link_04_name" value="link4_1" />
- <xacro:property name="link_05_name" value="link5_1" />
- <xacro:property name="link_06_name" value="link6_1" />
- <xacro:property name="joint_01_name" value="cadera_1" />
- <xacro:property name="joint_02_name" value="hombro_1" />
- <xacro:property name="joint_03_name" value="codo_1" />
- <xacro:property name="joint_04_name" value="mano_1" />
- <xacro:property name="joint_05_name" value="gripper0_1" />
- <xacro:property name="joint_06_name" value="gripper1_1" />
+ <xacro:property name="link_00_name" value="base_link" />
+ <xacro:property name="link_01_name" value="link1" />
+ <xacro:property name="link_02_name" value="link2" />
+ <xacro:property name="link_03_name" value="link3" />
+ <xacro:property name="link_04_name" value="link4" />
+ <xacro:property name="link_05_name" value="link5" />
+ <xacro:property name="link_06_name" value="link6" />
+ <xacro:property name="joint_01_name" value="cadera" />
+ <xacro:property name="joint_02_name" value="hombro" />
+ <xacro:property name="joint_03_name" value="codo" />
+ <xacro:property name="joint_04_name" value="mano" />
+ <xacro:property name="joint_05_name" value="gripper0" />
+ <xacro:property name="joint_06_name" value="gripper1" />
 </robot>

Commit message: Third

File: Intermedio/urdf/phantom_1.xacro (robot description, xacro)
@@ -14,8 +14,8 @@
  <property name="M_PI" value="3.14159" />
   <!-- Robot description -->
-  <link name="base_footprint"/>  <!-- Base link from Gazebo-->
+  <link name="world"/>  <!-- Base link from Gazebo-->
 	<!-- Joint to fix the base so it does not move-->
   <joint name="fixed" type="fixed">
-    <parent link="base_footprint"/>
+    <parent link="world"/>
     <child link="${link_00_name}"/>
   </joint>
@@ -141,8 +141,8 @@
   <!-- Plugin Gazebo -->
   <gazebo>
-     <plugin name="gazebo_ros_control" filename="libgazebo_ros_control.so">
-     <robotSimType>gazebo_ros_control/DefaultRobotHWSim</robotSimType>
- <legacyModeNS>true</legacyModeNS>
-     </plugin>
+    <plugin name="gazebo_ros_control" filename="libgazebo_ros_control.so">
+      <robotSimType>gazebo_ros_control/DefaultRobotHWSim</robotSimType>
+      <legacyModeNS>true</legacyModeNS>
+    </plugin>
   </gazebo>
 </robot>
